File: sailingRegattaTimer.kicad_sch (KiCad schematic)
At the start: 25 parts, among them J1 Power, J1-Red-1M1 Conn_01x02_Socket, J2 Digital/PWM, J2-Yel-2M1 Conn_01x02_Socket, J3 Analog, J3-Grn-3M1 J3-Grn-3M, J4 Digital/PWM, J4-Blu-5M1 J4-Blu-5M1, J5-5v-LED1 Conn_01x02_Socket, J6-Reset1 J6-Reset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

Commit message: added 12v input connector supplying voltage regulator
Parts:
- added J10-12v-In: Conn_01x02_Socket, Connector_PinSocket_2.54mm:PinSocket_1x02_P2.54mm_Vertical, symbol Connector:Conn_01x02_Socket
- renumbered D1 to D1-LED1
Connections:
- net GND: now also J10-12v-In.2 (Pin_2)
- net at J8-Pololu-VReg1.2 (Pin_2): now also J10-12v-In.1 (Pin_1)
Other:
- moved on the sheet: J8-Pololu-VReg1
Changed lines of the file:
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@@
+	)
+	(junction
+		(at 58.42 120.65)
+		(diameter 0)
+		(color 0 0 0 0)
 	)
 	(junction
@@
 	(wire
 		(pts
-			(xy 49.53 85.09) (xy 49.53 113.03)
+			(xy 49.53 85.09) (xy 49.53 120.65)
 		)
 		(stroke
@@
 	(wire
 		(pts
+			(xy 64.77 110.49) (xy 58.42 110.49)
+		)
+		(stroke
+			(width 0)
+			(type default)
+		)
+	)
+	(wire
+		(pts
 			(xy 68.58 60.96) (xy 68.58 73.66)
 		)
@@
 	(wire
 		(pts
-			(xy 45.72 115.57) (xy 45.72 81.28)
+			(xy 45.72 123.19) (xy 45.72 81.28)
 		)
 		(stroke
@@
 	(wire
 		(pts
+			(xy 58.42 110.49) (xy 58.42 120.65)
+		)
+		(stroke
+			(width 0)
+			(type default)
+		)
+	)
+	(wire
+		(pts
 			(xy 66.04 95.25) (xy 81.28 95.25)
 		)
@@
 	(wire
 		(pts
+			(xy 62.23 118.11) (xy 64.77 118.11)
+		)
+		(stroke
+			(width 0)
+			(type default)
+		)
+	)
+	(wire
+		(pts
+			(xy 58.42 120.65) (xy 64.77 120.65)
+		)
+		(stroke
+			(width 0)
+			(type default)
+		)
+	)
+	(wire
+		(pts
 			(xy 68.58 85.09) (xy 68.58 86.36)
 		)
@@
 	(wire
 		(pts
-			(xy 66.04 102.87) (xy 60.96 102.87)
+			(xy 60.96 102.87) (xy 66.04 102.87)
 		)
 		(stroke
@@
 	(wire
 		(pts
-			(xy 49.53 113.03) (xy 60.96 113.03)
+			(xy 49.53 120.65) (xy 58.42 120.65)
 		)
 		(stroke
@@
 	(wire
 		(pts
+			(xy 62.23 107.95) (xy 62.23 118.11)
+		)
+		(stroke
+			(width 0)
+			(type default)
+		)
+	)
+	(wire
+		(pts
 			(xy 176.53 63.5) (xy 189.23 63.5)
 		)
@@
 	(wire
 		(pts
-			(xy 60.96 115.57) (xy 45.72 115.57)
+			(xy 64.77 123.19) (xy 45.72 123.19)
 		)
 		(stroke
@@
 		(pts
 			(xy 176.53 83.82) (xy 176.53 93.98)
+		)
+		(stroke
+			(width 0)
+			(type default)
+		)
+	)
+	(wire
+		(pts
+			(xy 64.77 107.95) (xy 62.23 107.95)
 		)
 		(stroke
@@
 	(symbol
 		(lib_id "Connector:Conn_01x04_Socket")
-		(at 66.04 110.49 0)
+		(at 69.85 118.11 0)
 		(unit 1)
 		(exclude_from_sim no)
@@
 		(fields_autoplaced yes)
 		(property "Reference" "J8-Pololu-VReg1"
-			(at 67.31 110.4899 0)
+			(at 71.12 118.1099 0)
 			(effects
 				(font
@@
 		)
 		(property "Value" "Conn_01x04_Socket"
-			(at 67.31 113.0299 0)
+			(at 71.12 120.6499 0)
 			(effects
 				(font
@@
 		)
 		(property "Footprint" "Connector_PinSocket_2.54mm:PinSocket_1x04_P2.54mm_Vertical"
-			(at 66.04 110.49 0)
+			(at 69.85 118.11 0)
 			(effects
 				(font
@@
 		)
 		(property "Datasheet" "~"
-			(at 66.04 110.49 0)
+			(at 69.85 118.11 0)
 			(effects
 				(font
@@
 		)
 		(property "Description" "Generic connector, single row, 01x04, script generated"
-			(at 66.04 110.49 0)
+			(at 69.85 118.11 0)
 			(effects
 				(font
@@
 	(symbol
 		(lib_id "Connector:Conn_01x02_Socket")
+		(at 69.85 107.95 0)
+		(unit 1)
+		(exclude_from_sim no)
+		(in_bom yes)
+		(on_board yes)
+		(dnp no)
+		(fields_autoplaced yes)
+		(property "Reference" "J10-12v-In"
+			(at 71.12 109.2199 0)
+			(effects
+				(font
+					(size 1.27 1.27)
+				)
+				(justify left)
+			)
+		)
+		(property "Value" "Conn_01x02_Socket"
+			(at 71.12 110.4899 0)
+			(effects
+				(font
+					(size 1.27 1.27)
+				)
+				(justify left)
+				(hide yes)
+			)
+		)
+		(property "Footprint" "Connector_PinSocket_2.54mm:PinSocket_1x02_P2.54mm_Vertical"
+			(at 69.85 107.95 0)
+			(effects
+				(font
+					(size 1.27 1.27)
+				)
+				(hide yes)
+			)
+		)
+		(property "Datasheet" "~"
+			(at 69.85 107.95 0)
+			(effects
+				(font
+					(size 1.27 1.27)
+				)
+				(hide yes)
+			)
+		)
+		(property "Description" "Generic connector, single row, 01x02, script generated"
+			(at 69.85 107.95 0)
+			(effects
+				(font
+					(size 1.27 1.27)
+				)
+				(hide yes)
+			)
+		)
+		(pin "1"
+		)
+		(pin "2"
+		)
+		(instances
+			(project "sailingRegattaTimer"
+				(path "/e63e39d7-6ac0-4ffd-8aa3-1841a4541b55"
+					(reference "J10-12v-In")
+					(unit 1)
+				)
+			)
+		)
+	)
+	(symbol
+		(lib_id "Connector:Conn_01x02_Socket")
 		(at 176.53 146.05 0)
 		(unit 1)
@@
 		(dnp no)
 		(fields_autoplaced yes)
-		(property "Reference" "D1"
+		(property "Reference" "D1-LED1"
 			(at 168.5925 121.92 0)
 			(effects
@@
 					(size 1.27 1.27)
 				)
+				(hide yes)
 			)
 		)
@@
 			(project ""
 				(path "/e63e39d7-6ac0-4ffd-8aa3-1841a4541b55"
-					(reference "D1")
+					(reference "D1-LED1")
 					(unit 1)
 				)

Commit message: 20250423-095156 checkin based on latest board check and changes to support automated testing
Parts:
- renumbered J10-12v-In to J10-12v-In1
Changed lines of the file:
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@@
 		(dnp no)
 		(fields_autoplaced yes)
-		(property "Reference" "J10-12v-In"
+		(property "Reference" "J10-12v-In1"
 			(at 71.12 109.2199 0)
 			(effects
@@
 			(project "sailingRegattaTimer"
 				(path "/e63e39d7-6ac0-4ffd-8aa3-1841a4541b55"
-					(reference "J10-12v-In")
+					(reference "J10-12v-In1")
 					(unit 1)
 				)

Commit message: save incremental work
Parts:
- added TM1637-+5-GND, TM1637-DIO-CLK: Conn_01x02_Socket, Connector_PinSocket_2.54mm:PinSocket_1x02_P2.54mm_Vertical, symbol Connector:Conn_01x02_Socket
- D1-LED1: footprint LED_THT:LED_D1.8mm_W1.8mm_H2.4mm_Horizontal_O1.27mm_Z1.6mm -> LED_THT:LED_D3.0mm
Connections:
- net *3: now also TM1637-DIO-CLK.2 (Pin_2)
- net *5: now also TM1637-DIO-CLK.1 (Pin_1)
- net +5V: now also TM1637-+5-GND.1 (Pin_1)
- net GND: now also TM1637-+5-GND.2 (Pin_2)
- net VCC: no longer J1.8 (Pin_8)
- net IOREF: no longer names the net of J1.2 (Pin_2)
- net ~{RESET}: no longer names the net of J1.3 (Pin_3), J6-Reset1.1 (Pin_1), SW5-Reset1.1
Other:
- note added: "IOREF"
- note added: "RESET"
- moved on the sheet: J1, J1-Red-1M1, J10-12v-In1, J2-Yel-2M1, J3, J3-Grn-3M1, J5-5v-LED1, J6-Reset1, J7-Ext-Buz1, J8-Pololu-VReg1, J9-Relay1, R1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

Commit message: incremental save, updated schematic, schematic image and pcb initial
Parts:
- removed J1: Power, Connector_PinSocket_2.54mm:PinSocket_1x08_P2.54mm_Vertical, symbol Connector_Generic:Conn_01x08
- removed J2: Digital/PWM, Connector_PinSocket_2.54mm:PinSocket_1x10_P2.54mm_Vertical, symbol Connector_Generic:Conn_01x10
- removed J3: Analog, Connector_PinSocket_2.54mm:PinSocket_1x06_P2.54mm_Vertical, symbol Connector_Generic:Conn_01x06
- removed J4: Digital/PWM, Connector_PinSocket_2.54mm:PinSocket_1x08_P2.54mm_Vertical, symbol Connector_Generic:Conn_01x08
- added A1: Arduino_UNO_R3, Module:Arduino_UNO_R3, symbol MCU_Module:Arduino_UNO_R3
- renumbered TM1637-+5-GND to TM1637+5-GND1, TM1637-DIO-CLK to TM1637-CLK-DIO1
Connections:
- net at J6-Reset1.1 (Pin_1), SW5-Reset1.1: now also A1.3 (~{RESET})
- net *3: no longer names the net of TM1637-CLK-DIO1.2 (Pin_2)
- net *3: now also A1.20 (D5)
- net *5: no longer names the net of TM1637-CLK-DIO1.1 (Pin_1)
- net *5: now also A1.18 (D3)
- net 12: no longer names the net of J4-Blu-5M1.2 (Pin_2), R4.1, SW4-Blu-5M1.2
- net 12: now also A1.27 (D12)
- net 2: no longer names the net of J1-Red-1M1.2 (Pin_2), R1.1, SW1-Red-1M1.2
- net 2: now also A1.17 (D2)
- net 4: no longer names the net of BZ1.1 (+), D1-LED1.2 (A), J7-Ext-Buz1.1 (Pin_1)
- net 4: now also A1.19 (D4)
- net 7: no longer names the net of J2-Yel-2M1.2 (Pin_2), R2.1, SW2-Yel-2M1.2
- net 7: now also A1.22 (D7)
- net 8: no longer names the net of J3-Grn-3M1.2 (Pin_2), R3.1, SW3-Grn-3M1.2
- net 8: now also A1.23 (D8)
- net VCC: no longer names the net of J8-Pololu-VReg1.4 (Pin_4)
- net VCC: now also A1.8 (VIN)
- no-connect marks 1 -> 0
Other:
- note removed: "IOREF"
- note removed: "RESET"
- moved on the sheet: BZ1, D1-LED1, J1-Red-1M1, J10-12v-In1, J2-Yel-2M1, J3-Grn-3M1, J4-Blu-5M1, J5-5v-LED1, J6-Reset1, J7-Ext-Buz1, J8-Pololu-VReg1, J9-Relay1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

Commit message: incremental save updated schematic and pcb
Connections:
- net +5V: now also A1.5 (+5V)
- net GND: now also A1.29 (GND), A1.6 (GND), A1.7 (GND)
Other:
- moved on the sheet: J4-Blu-5M1, SW2-Yel-2M1, SW3-Grn-3M1

Commit message: remove production files, update schematic and pcb
Parts:
- A1: footprint Module:Arduino_UNO_R3 -> rt-uno:rt-Arduino_UNO_R3
- R1, R2, R3, R4: value ~ -> R; footprint Resistor_THT:R_Axial_DIN0309_L9.0mm_D3.2mm_P2.54mm_Vertical -> Resistor_THT:R_Axial_DIN0204_L3.6mm_D1.6mm_P1.90mm_Vertical

Commit message: updated images and one resistor footprint so it matched the others
Parts:
- R5: footprint Resistor_THT:R_Axial_DIN0309_L9.0mm_D3.2mm_P2.54mm_Vertical -> Resistor_THT:R_Axial_DIN0204_L3.6mm_D1.6mm_P1.90mm_Vertical
Changed lines of the file:
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@@
 			)
 		)
-		(property "Footprint" "Resistor_THT:R_Axial_DIN0309_L9.0mm_D3.2mm_P2.54mm_Vertical"
+		(property "Footprint" "Resistor_THT:R_Axial_DIN0204_L3.6mm_D1.6mm_P1.90mm_Vertical"
 			(at 177.292 134.62 90)
 			(effects

Commit message: incremental save
Parts:
- A1: footprint rt-uno:rt-Arduino_UNO_R3 -> Module:Arduino_UNO_R3
Changed lines of the file:
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@@
 			)
 		)
-		(property "Footprint" "rt-uno:rt-Arduino_UNO_R3"
+		(property "Footprint" "Module:Arduino_UNO_R3"
 			(at 189.23 87.63 0)
 			(effects
