File: sailingRegattaTimer.kicad_sch (KiCad schematic)
At the start: 25 parts, among them J1-Red-1M1 Conn_01x02_Socket, J10-12v-In1 Conn_01x02_Socket, J2-Yel-2M1 Conn_01x02_Socket, J3-Grn-3M1 J3-Grn-3M, J4-Blu-5M1 J4-Blu-5M1, J5-5v-LED1 Conn_01x02_Socket, J6-Reset1 J6-Reset, J7-Ext-Buz1 Conn_01x02_Socket, J8-Pololu-VReg1 Conn_01x04_Socket, J9-Relay1 Conn_01x03_Socket

Commit message: incremental save
Parts:
- A1: footprint Module:Arduino_UNO_R3 -> KiCad-Library:Arduino_UNO_R3
Changed lines of the file:
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@@
 			)
 		)
-		(property "Footprint" "Module:Arduino_UNO_R3"
+		(property "Footprint" "KiCad-Library:Arduino_UNO_R3"
 			(at 189.23 87.63 0)
 			(effects

Commit message: Revert "incremental save"
This reverts commit 1c0ff86f2212df186ba7f97aef935cadcedda2ad.
Parts:
- A1: footprint KiCad-Library:Arduino_UNO_R3 -> Module:Arduino_UNO_R3
Changed lines of the file:
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@@
 			)
 		)
-		(property "Footprint" "KiCad-Library:Arduino_UNO_R3"
+		(property "Footprint" "Module:Arduino_UNO_R3"
 			(at 189.23 87.63 0)
 			(effects
